Commit message: Remove unecessary files + update materials

File: urdf/materials.urdf.xacro (robot description, xacro)
@@ -32,3 +32,15 @@
     <color rgba="0.96 0.88 0.14 1.0"/>
   </material>
+  <material name="Black">
+    <color rgba="0.0 0.0 0.0 1.0"/>
+  </material>
+  <material name="Orange">
+    <color rgba="1.0 0.6 0.0 1.0"/>
+  </material>
+  <material name="pal/Orange">
+    <color rgba="0.91373 0.61568 0.29411 1.0"/>
+  </material>
+  <material name="pal/DarkGrey">
+    <color rgba="0.29804 0.29804 0.29804 1"/>
+  </material>
 </robot>

Commit message: Add new color and adapt Orange

File: urdf/materials.urdf.xacro (robot description, xacro)
@@ -35,6 +35,9 @@
     <color rgba="0.0 0.0 0.0 1.0"/>
   </material>
+  <material name="FlatBlack">
+    <color rgba="0.09 0.09 0.09 1.0"/>
+  </material>
   <material name="Orange">
-    <color rgba="1.0 0.6 0.0 1.0"/>
+    <color rgba="1.0 0.487 0.0 1.0"/>
   </material>
   <material name="pal/Orange">
